File: kicad_test.kicad_pcb (KiCad board)
At the start: 2 copper layers, 1 part, among them U1 IR4302

Commit message: test
Routing:
- net (no net): track 0.00 -> 4.87 mm
Changed lines of the file:
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@@
     )
   )
+  (segment (start 175.9885 72.36) (end 176.56 72.36) (width 0.2) (layer "F.Cu") (net 0))
+  (segment (start 177.8 71.12) (end 180.34 71.12) (width 0.2) (layer "F.Cu") (net 0))
+  (segment (start 176.56 72.36) (end 177.8 71.12) (width 0.2) (layer "F.Cu") (net 0))
 )
